File: kicad/2_nodes_3_hid/2_nodes_3_hid.kicad_sch (KiCad schematic)
At the start: 16 parts

Commit message: Add schematic and pcb design for 2 nodes with 3 hid and 3 hid with 3 nodes
Parts:
- added HID_DEV_3: USB_A, Connector_USB:USB_A_Molex_67643_Horizontal, symbol Connector:USB_A
- added USB_C3: 10 µF, Capacitor_SMD:C_1206_3216Metric_Pad1.33x1.80mm_HandSolder, symbol Device:C
- added USB_PD_DM3, USB_PD_DP3: 15K, Resistor_SMD:R_1206_3216Metric_Pad1.30x1.75mm_HandSolder, symbol Device:R
- added USB_R_DM3, USB_R_DP3: 22, Resistor_SMD:R_1206_3216Metric_Pad1.30x1.75mm_HandSolder, symbol Device:R
Connections:
- net GND: now also HID_DEV_3.4 (GND), HID_DEV_3.SH (Shield), USB_C3.1, USB_PD_DM3.1, USB_PD_DP3.2
- net vsys: now also HID_DEV_3.1 (VBUS), USB_C3.2
- net usb_3_d-: now reaches Controller1.14 (GPIO10)
- net usb_3_d-: now also USB_R_DM3.2
- net usb_3_d+: now reaches Controller1.15 (GPIO11)
- net usb_3_d+: now also USB_R_DP3.2
- new net: HID_DEV_3.3 (D+), USB_PD_DP3.1, USB_R_DP3.1
- new net: HID_DEV_3.2 (D-), USB_PD_DM3.2, USB_R_DM3.1
Other:
- title: KVM Switch - 2 Nodes - 2 HID -> KVM Switch - 2 Nodes - 3 HID
